Commit message: add original urdf file to the package

File: irb2600/abb_irb2600_support/urdf/irb2600_12_165.xacro (robot description, xacro)
@@ -3,14 +3,3 @@
   <xacro:include filename="$(find abb_irb2600_support)/urdf/irb2600_12_165_macro.xacro"/>
   <xacro:abb_irb2600_12_165 prefix=""/>
-  <xacro:arg name="use_nominal_extrinsics" default="true" />
-  <xacro:arg name="add_plug" default="true" />
-  <xacro:arg name="use_mesh" default="true" />
-  <xacro:include filename="$(find tool_description)/urdf/draping_tool.urdf.xacro" />
-  <!-- <xacro:include filename="$(find realsense2_description)/urdf/_d415.urdf.xacro" /> -->
-  <xacro:draping_tool parent="camera_mount" use_nominal_extrinsics="$(arg use_nominal_extrinsics)" use_mesh="$(arg use_mesh)">
-    <origin xyz="0 0 0" rpy="0 -1.57 -0.61"/>
-  </xacro:draping_tool>
-  <!-- <xacro:sensor_d415 parent="camera_mount" use_nominal_extrinsics="$(arg use_nominal_extrinsics)" use_mesh="$(arg use_mesh)">
-    <origin xyz="-0.004 0.0 0.031" rpy="0 -1.57 0"/>
-  </xacro:sensor_d415> -->
 </robot>

File: irb2600/abb_irb2600_support/urdf/irb2600_12_165_macro_rishi.xacro (robot description, xacro)
@@ -111,5 +111,5 @@
       </collision>
     </link>
-    <!-- Joints -->
+    <!-- Joints - Rishi modified axis 1 (maybe axis 3 also) of abb so it doesn't swing around-->
     <joint name="${prefix}joint_1" type="revolute">
       <origin xyz="0 0 0.445" rpy="0 0 0" />
@@ -117,5 +117,5 @@
       <child link="${prefix}link_1" />
       <axis xyz="0 0 1" />
-      <limit lower="-3.14159" upper="3.14159" effort="0" velocity="3.054" />
+      <limit lower="-0.7" upper="3.0" effort="0" velocity="3.054" />
     </joint>
     <joint name="${prefix}joint_2" type="revolute">
@@ -138,5 +138,5 @@
       <child link="${prefix}link_4" />
       <axis xyz="1 0 0" />
-      <limit lower="-6.981" upper="6.981" effort="0" velocity="6.283" />
+      <limit lower="1.4" upper="5.0" effort="0" velocity="6.283" />
     </joint>
     <joint name="${prefix}joint_5" type="revolute">
@@ -175,4 +175,48 @@
       <child link="${prefix}tool0" />
     </joint>
+    <link name="camera_mount">
+      <visual>
+      <geometry>
+          <mesh filename="package://system/database/meshes/camera_mount.stl"
+              scale="1 1 1"/>
+      </geometry>
+      <material name="ABS" >
+          <color rgba="0.5 0.5 0.5 1.0" />
+          </material>
+      </visual>
+      <collision>
+        <origin xyz="0 0 0" rpy="0 0 0" />
+        <geometry>
+          <mesh filename="package://system/database/meshes/camera_mount.stl" />
+        </geometry>
+      </collision>
+    </link>
+    <joint type="fixed" name="mount_joint">
+        <origin xyz="0 0 0" rpy="0 0 0"/>
+        <parent link="${prefix}tool0"/>
+        <child link="camera_mount"/>
+    </joint>
+    <link name="mould">
+      <visual>
+        <origin xyz="0.626565 0.631265 0.140994" rpy="0.0033 -0.1027 2.88" />
+        <geometry>
+          <mesh filename="package://system/database/meshes/mould.stl" scale="0.001 0.001 0.001"/>
+        </geometry>
+        <material name="ABS" >
+          <color rgba="0.5 0.5 0.5 1.0" />
+        </material>
+      </visual>
+      <collision>
+        <origin xyz="0.626565 0.631265 0.140994" rpy="0.0033 -0.1027 2.88" />
+        <geometry>
+          <mesh filename="package://system/database/meshes/mould.stl" scale="0.001 0.001 0.001"/>
+        </geometry>
+      </collision>
+    </link>
+    <joint type="fixed" name="mould_joint">
+        <origin xyz="0 0 0" rpy="0 0 0"/>
+        <parent link="${prefix}base_link"/>
+        <child link="mould"/>
+    </joint>
   </xacro:macro>
 </robot>
